Commit message: Mirrored changes to URDF.

File: iai_gazebo_visibility_mover/urdf/boxy_description.urdf (robot description, URDF)
Before this commit: robot boxy_description, 72 links, 71 joints
Joints:
- joint left_gripper_anterior_gripper_joint: origin xyz=0 0 0 rpy=0 0 0.78539816339 -> xyz=0 0 0 rpy=0 0 2.3562
- joint neck_adapter_ur3_in_joint: origin xyz=0.214 -0.227 1.48 rpy=0 0 0 -> xyz=0.175 -0.227 1.48 rpy=0 0 0

Commit message: Corrected colouring of simulation boxy.

File: iai_gazebo_visibility_mover/urdf/boxy_description.urdf (robot description, URDF)
Before this commit: robot boxy_description, 72 links, 71 joints
Links:
- removed link base_link
- added link boxy_base_link, mass 70.0210745907357; collision mesh filename=package://iai_boxy_base/meshes/base_link_simple.STL; visual mesh filename=package://iai_boxy_base/meshes/base_link.dae
Joints:
- joint base_footprint_joint: child base_link -> boxy_base_link
- joint laser_reference_back_joint: parent base_link -> boxy_base_link
- joint laser_reference_front_joint: parent base_link -> boxy_base_link
- joint neck_adapter_ur3_in_joint: parent base_link -> boxy_base_link
- joint shoulder_kinect_joint: parent base_link -> boxy_base_link
- joint torso_joint: parent base_link -> boxy_base_link
- joint triangle_base_joint: parent base_link -> boxy_base_link
